Commit message: update

File: ros2_ws/install/robot_description/share/robot_description/description/robot_core.xacro (robot description, xacro)
@@ -13,4 +13,7 @@
     <material name="black">
         <color rgba="0 0 0 1"/>
+    </material>
+    <material name="red">
+    <color rgba="1 0 0 1"/>
     </material>
     <!-- BASE LINK -->
